File: hw/IMU_module.sch (EAGLE design)
At the start: 42 parts, among them J1 GROVE-4P-2.0-3470130P1, J2 GROVE-4P-2.0-3470130P1, X1 53047-06

Commit message: Renamed gyro DRDY signal and updated makefile
Connections:
- net GYRO_INT2 renamed GYRO_DRDY
Changed lines of the file:
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@@
 </segment>
 </net>
-<net name="GYRO_INT2" class="0">
+<net name="GYRO_DRDY" class="0">
 <segment>
 <wire x1="175.26" y1="228.6" x2="172.72" y2="228.6" width="0.1524" layer="91"/>
